File: PCB_Design/Drone_Chassis/Drone_Chassis.kicad_sch (KiCad schematic)
At the start: 0 parts

Commit message: FC_Desing_Start
Parts:
- added BT1: Battery_Cell, Connector_Molex:Molex_Micro-Fit_3.0_43045-0212_2x01_P3.00mm_Vertical, symbol Device:Battery_Cell
- added C1: 10u, Capacitor_SMD:C_0402_1005Metric, symbol Device:C
- added C11, C12: 22U, Capacitor_SMD:C_0603_1608Metric, symbol Device:C
- added C2: 1u, Capacitor_SMD:C_0402_1005Metric, symbol Device:C
- added C3: 100n, Capacitor_SMD:C_0402_1005Metric, symbol Device:C
- added D1, D2, D3: LED, LED_SMD:LED_0603_1608Metric, symbol Device:LED
- added J9: USB_C_Receptacle_USB2.0_16P_ESP32, Connector_USB:USB_C_Receptacle_GCT_USB4105-xx-A_16P_TopMnt_Horizontal, symbol Connector:USB_C_Receptacle_USB2.0_16P
- added M1: M1_Motor_PWM, Jumper:SolderJumper-3_P1.3mm_Bridged2Bar12_Pad1.0x1.5mm, symbol Mechanical:MountingHole_Pad_MP
- added M2: M2_Motor_PWM, Jumper:SolderJumper-3_P1.3mm_Bridged2Bar12_Pad1.0x1.5mm, symbol Mechanical:MountingHole_Pad_MP
- added M3: M3_Motor_PWM, Jumper:SolderJumper-3_P1.3mm_Bridged2Bar12_Pad1.0x1.5mm, symbol Mechanical:MountingHole_Pad_MP
- added M4: M4_Motor_PWM, Jumper:SolderJumper-3_P1.3mm_Bridged2Bar12_Pad1.0x1.5mm, symbol Mechanical:MountingHole_Pad_MP
- added R1: 0k2, Resistor_SMD:R_0402_1005Metric, symbol Device:R
- added R14, R15, R17, R2, R3: 1k5, Resistor_SMD:R_0603_1608Metric, symbol Device:R
- added R16: 0k4, Resistor_SMD:R_0603_1608Metric, symbol Device:R
- added R18, R19, R20, R21, R22: 10k, Resistor_SMD:R_0603_1608Metric, symbol Device:R
- added R4, R5: 1k5, Resistor_SMD:R_0402_1005Metric, symbol Device:R
- added R6, R7: 5k1, Resistor_SMD:R_0603_1608Metric, symbol Device:R
- added SW1, SW2: SW_Push, Button_Switch_THT:SW_PUSH_6mm_H4.3mm, symbol Switch:SW_Push
- added U1: TP4056-42-ESOP8, Package_SO:SOIC-8-1EP_3.9x4.9mm_P1.27mm_EP2.41x3.3mm_ThermalVias, symbol Battery_Management:TP4056-42-ESOP8
- added U2: ESP32-S3-WROOM-1, RF_Module:ESP32-S3-WROOM-1, symbol RF_Module:ESP32-S3-WROOM-1
- added U3: AMS1117-3.3, Package_TO_SOT_SMD:SOT-223-3_TabPin2, symbol Regulator_Linear:AMS1117-3.3
- added U4: MPU-9250, Sensor_Motion:InvenSense_QFN-24_3x3mm_P0.4mm, symbol Sensor_Motion:MPU-9250
- added U5: BMP280, Package_LGA:Bosch_LGA-8_2x2.5mm_P0.65mm_ClockwisePinNumbering, symbol Sensor_Pressure:BMP280
- added U6: INA219AxD, Package_SO:SOIC-8_3.9x4.9mm_P1.27mm, symbol Sensor_Energy:INA219AxD
Connections:
- new net: R14.1, R15.1, R16.1, U1.4 (V_{CC}), U1.8 (CE)
- new net: D2.2 (A), R14.2
- new net: R18.2, U1.1 (TEMP)
- new net: R17.2, U1.2 (PROG)
- new net: D3.1 (K), U1.6 (~{STDBY})
- new net: D2.1 (K), U1.7 (~{CHRG})
- new net: R5.1, U6.3 (SDA)
- new net: R4.1, U6.4 (SCL)
- new net: R1.2, U6.7 (IN-)
- new net: R1.1, U6.8 (IN+)
- new net: D1.1 (K), R3.1
- new net: R19.2, SW1.2, U2.3 (EN)
- new net: J9.B5 (CC2), R7.1
- new net: R20.2, SW2.2, U2.27 (IO0)
- new net: D3.2 (A), R15.2
- new net: J9.A5 (CC1), R6.1
- new net +3.3V: C12.1, C2.1, C3.1, D1.2 (A), R19.1, R2.1, R20.1, R4.2, R5.2, U2.2 (3V3), U3.2 (VO), U6.5 (VS)
- new net BAT+: BT1.1 (+), C1.1, R21.2, U1.5 (BAT)
- new net GND: BT1.2 (-), C1.2, C11.2, C12.2, C2.2, C3.2, J9.A1 (GND), J9.A12 (GND), J9.B1 (GND), J9.B12 (GND), R17.1, R18.1, R22.1, R3.2, R6.2, R7.2, SW1.1, SW2.1, U1.3 (GND), U1.9 (EPAD), U2.1 (GND), U2.40 (GND), U2.41 (GND), U3.1 (GND), U6.1 (A1), U6.2 (A0), U6.6 (GND)
- new net MCU_IN_BAT: R21.1, R22.2, U2.31 (IO38)
- new net USB_D+: J9.A6 (D+), J9.B6 (D+), R2.2, U2.14 (USB_D+)
- new net USB_D-: J9.A7 (D-), J9.B7 (D-), U2.13 (USB_D-)
- new net VBUS: C11.1, J9.A4 (VBUS), J9.A9 (VBUS), J9.B4 (VBUS), J9.B9 (VBUS), R16.2, U3.3 (VI)
- no-connect marks 0 -> 35
