File: PCB_Design/Drone_Controller/Drone_Controller.kicad_sch (KiCad schematic)
At the start: 40 parts, among them J1 Conn_01x03_Pin, J2 Conn_01x08_Socket, J9 USB_C_Receptacle_USB2.0_16P_E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, SW1 SW_Push, SW2 SW_Push, SW3 SW_Push, SW4 SW_Push, SW5 SW_Push, SW6 SW_Push, U1 TP4056-42-ESOP8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

Commit message: PCB_V1_Final
Parts:
- BT1: footprint Connector_Molex:Molex_Micro-Fit_3.0_43045-0212_2x01_P3.00mm_Vertical -> Connector_JST:JST_PH_S2B-PH-SM4-TB_1x02-1MP_P2.00mm_Horizontal
Other:
- note added: "@EmrecanBL"
- note added: "ANALOG_STICKS"
- note added: "BATTERY MESUARING"
- note added: "LCD_SOCKET"
- note added: "MCU(ESP32-WROOM-1)"
- note added: "POWER_MANAGEMENT"
- note added: "USB & USB-CONNECTIONS"
- note added: "USER_BUTON"
- moved on the sheet: BT1, J2
