File: PCB_Design/Drone_Controller/Drone_Controller.kicad_pcb (KiCad board)
At the start: 2 copper layers, 115.7 x 43.1 mm, 40 parts, among them J1 Conn_01x03_Pin, J2 Conn_01x08_Socket, J9 USB_C_Receptacle_USB2.0_16P_E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, SW1 SW_Push, SW2 SW_Push, SW3 SW_Push, SW4 SW_Push, SW5 SW_Push, SW6 SW_Push, U1 TP4056-42-ESOP8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

Commit message: PCB_V1_Final
Parts:
- BT1: moved to B.Cu
- turned BT1 to 180 degrees

Commit message: Update
Other:
- board text added: "@EmrecanBL"
Changed lines of the file:
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@@
 		(layer "Edge.Cuts")
+	)
+	(gr_text "@EmrecanBL"
+		(at 80.53 76.4 0)
+		(layer "B.SilkS")
+		(effects
+			(font
+				(size 2 2)
+				(thickness 0.1)
+			)
+			(justify left bottom mirror)
+		)
 	)
 	(segment
