File: PCB_Design/Drone_Chassis/Bottom-Stack/Bottom-Stack.kicad_pcb (KiCad board)
At the start: 4 copper layers, 88.8 x 78.8 mm, 42 parts, among them J1 Conn_02x05_Top_Bottom, J2 ESC_M1_Connector, J3 ESC_M2_Connector, J4 ESC_M3_Connector, J5 ESC_M4_Connector, J6 Conn_02x05_Top_Bottom, J7 Battery_Connector, U1 TP4056-42-ESOP8, U2 VL53L1CXV0FY1, U3 AMS1117-3.3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

Commit message: Update
Other:
- board text added: "@EmrecanBL"
Changed lines of the file:
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@@
 		(layer "Edge.Cuts")
+	)
+	(gr_text "@EmrecanBL"
+		(at 55.61 46.435 180)
+		(layer "B.SilkS")
+		(effects
+			(font
+				(size 2 2)
+				(thickness 0.1)
+			)
+			(justify left bottom mirror)
+		)
 	)
 	(segment
