File: PCB_Design/Drone_Chassis/Middle-Stack/Drone_Chassis.kicad_pcb (KiCad board)
At the start: 4 copper layers, 39 x 39 mm, 43 parts, among them J1 Conn_02x05_Top_Bottom, J6 Conn_02x05_Top_Bottom, J9 USB_C_Receptacle_USB2.0_16P_E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, SW1 SW_Push, SW2 SW_Push, U1 SAM-M10Q, U2 ESP32-S3-WROOM-1, U4 MPU-9250, U5 BMP280

Commit message: Update
Other:
- board text added: "@EmrecanBL"
Changed lines of the file:
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@@
 		(layer "Edge.Cuts")
+	)
+	(gr_text "@EmrecanBL"
+		(at 51.54 27.04 0)
+		(layer "B.SilkS")
+		(effects
+			(font
+				(size 2 2)
+				(thickness 0.1)
+			)
+			(justify left bottom mirror)
+		)
 	)
 	(segment
